Commit message: rename package and files

File: urdf/robot.xacro (robot description, xacro)
@@ -1,5 +1,5 @@
 <?xml version='1.0'?>
-<robot name="my_robot" xmlns:xacro="http://www.ros.org/wiki/xacro">
-<xacro:include filename="$(find my_robot)/urdf/my_robot.gazebo" />
+<robot name="robot" xmlns:xacro="http://www.ros.org/wiki/xacro">
+<xacro:include filename="$(find gazebo_simulation)/urdf/robot.gazebo" />
   <gazebo reference="chassis">
     <material>Gazebo/White</material>
@@ -178,5 +178,5 @@
       <origin xyz="0 0 0" rpy=" 0 0 0"/>
       <geometry>
-        <mesh filename="package://my_robot/meshes/hokuyo.dae"/>
+        <mesh filename="package://gazebo_simulation/meshes/hokuyo.dae"/>
       </geometry>
     </visual>

Commit message: Add IMU, still need to test if the sensor works

File: urdf/robot.xacro (robot description, xacro)
@@ -188,3 +188,29 @@
     <axis xyz="0 1 0" rpy="0 0 0"/>
   </joint>
+  <!-- IMU -->
+    <link name="imu_link">
+    <inertial>
+      <mass value="0.001"/>
+      <origin rpy="0 0 0" xyz="0 0 0"/>
+      <inertia ixx="0.0001" ixy="0" ixz="0" iyy="0.000001" iyz="0" izz="0.0001"/>
+    </inertial>
+    <visual>
+      <origin rpy="0 0 0" xyz="0 0 0"/>
+      <geometry>
+        <box size="0.001 0.001 0.001"/>
+      </geometry>
+    </visual>
+    <collision>
+      <origin rpy="0 0 0" xyz="0 0 0"/>
+      <geometry>
+        <box size=".001 .001 .001"/>
+      </geometry>
+    </collision>
+  </link>
+  <joint name="imu_joint" type="fixed">
+    <axis xyz="1 0 0"/> <!-- 0 1 0 -->
+    <origin xyz="0 0 0.19"/>
+    <parent link="chassis"/>
+    <child link="imu_link"/>
+  </joint>
 </robot>

Commit message: switch to 4 wheels

File: urdf/robot.xacro (robot description, xacro)
@@ -8,10 +8,17 @@
     <material>Gazebo/Grey</material>
   </gazebo>
-  <gazebo reference="left_wheel">
-    <material>Gazebo/Black</material>
-  </gazebo>
-  <gazebo reference="right_wheel">
-    <material>Gazebo/Black</material>
-  </gazebo>
+  <gazebo reference="left_wheel_front">
+    <material>Gazebo/Black</material>
+  </gazebo>
+  <gazebo reference="right_wheel_front">
+    <material>Gazebo/Black</material>
+  </gazebo>
+  <gazebo reference="left_wheel_back">
+    <material>Gazebo/Black</material>
+  </gazebo>
+  <gazebo reference="right_wheel_back">
+    <material>Gazebo/Black</material>
+  </gazebo>
+  <!-- ROBOT description -->
   <link name="robot_footprint"></link>
   <joint name="robot_footprint_joint" type="fixed">
@@ -43,91 +50,134 @@
       </geometry>
     </visual>
-    <collision name='back_caster_collision'>
-      <origin xyz="-0.15 0 -0.05" rpy=" 0 0 0"/>
-      <geometry>
-        <sphere radius="0.0499"/>
-      </geometry>
-    </collision>
-    <visual name='back_caster_visual'>
-      <origin xyz="-0.15 0 -0.05" rpy=" 0 0 0"/>
-      <geometry>
-        <sphere radius="0.05"/>
-      </geometry>
-    </visual>
-    <collision name='front_caster_collision'>
-      <origin xyz="0.15 0 -0.05" rpy=" 0 0 0"/>
-      <geometry>
-        <sphere radius="0.0499"/>
-      </geometry>
-    </collision>
-    <visual name='front_caster_visual'>
-      <origin xyz="0.15 0 -0.05" rpy=" 0 0 0"/>
-      <geometry>
-        <sphere radius="0.05"/>
-      </geometry>
-    </visual>
-  </link>
-  <link name='left_wheel'>
-    <inertial>
-      <mass value="5.0"/>
-      <origin xyz="0.0 0 0" rpy=" 0 1.5707 1.5707"/>
-      <inertia
-          ixx="0.1" ixy="0" ixz="0"
-          iyy="0.1" iyz="0"
-          izz="0.1"
-      />
-    </inertial>
-    <collision name='left_wheel_collision'>
-      <origin xyz="0 0 0" rpy=" 0 1.5707 1.5707"/>
-      <geometry>
-        <cylinder length="0.05" radius="0.1"/>
-      </geometry>
-    </collision>
-    <visual name='left_wheel_visual'>
-      <origin xyz="0 0 0" rpy=" 0 1.5705 1.5707"/>
-      <geometry>
-        <cylinder length="0.05" radius="0.1"/>
-      </geometry>
-    </visual>
-  </link>
-  <joint type="continuous" name="left_wheel_hinge">
-    <origin xyz="0.0 0.15 0" rpy="0 0 0"/>
-    <child link="left_wheel"/>
-    <parent link="chassis"/>
-    <axis xyz="0 1 0" rpy="0 0 0"/>
-    <limit effort="10000" velocity="1000"/>
-    <dynamics damping="1.0" friction="1.0"/>
-  </joint>
-  <link name='right_wheel'>
-    <inertial>
-      <mass value="5.0"/>
-      <origin xyz="0.0 0 0" rpy=" 0 1.5707 1.5707"/>
-      <inertia
-          ixx="0.1" ixy="0" ixz="0"
-          iyy="0.1" iyz="0"
-          izz="0.1"
-      />
-    </inertial>
-    <collision name='right_wheel_collision'>
-      <origin xyz="0 0 0" rpy=" 0 1.5707 1.5707"/>
-      <geometry>
-        <cylinder length="0.05" radius="0.1"/>
-      </geometry>
-    </collision>
-    <visual name='right_wheel_visual'>
-      <origin xyz="0 0 0" rpy=" 0 1.5705 1.5707"/>
-      <geometry>
-        <cylinder length="0.05" radius="0.1"/>
-      </geometry>
-    </visual>
-  </link>
-  <joint type="continuous" name="right_wheel_hinge">
-    <origin xyz="0.0 -0.15 0" rpy="0 0 0"/>
-    <child link="right_wheel"/>
-    <parent link="chassis"/>
-    <axis xyz="0 1 0" rpy="0 0 0"/>
-    <limit effort="10000" velocity="1000"/>
-    <dynamics damping="1.0" friction="1.0"/>
-  </joint>
+  </link>
+  <!-- Left wheel front -->
+  <link name='left_wheel_front'>
+    <inertial>
+      <mass value="5.0"/>
+      <origin xyz="0.0 0 0" rpy=" 0 1.5707 1.5707"/>
+      <inertia
+          ixx="0.1" ixy="0" ixz="0"
+          iyy="0.1" iyz="0"
+          izz="0.1"
+      />
+    </inertial>
+    <collision name='left_wheel_front_collision'>
+      <origin xyz="0 0 0" rpy=" 0 1.5707 1.5707"/>
+      <geometry>
+        <cylinder length="0.05" radius="0.1"/>
+      </geometry>
+    </collision>
+    <visual name='left_wheel_front_visual'>
+      <origin xyz="0 0 0" rpy=" 0 1.5705 1.5707"/>
+      <geometry>
+        <cylinder length="0.05" radius="0.1"/>
+      </geometry>
+    </visual>
+  </link>
+  <joint type="continuous" name="left_wheel_front_hinge">
+    <origin xyz="0.15 0.15 0" rpy="0 0 0"/>
+    <child link="left_wheel_front"/>
+    <parent link="chassis"/>
+    <axis xyz="0 1 0" rpy="0 0 0"/>
+    <limit effort="10000" velocity="1000"/>
+    <dynamics damping="1.0" friction="1.0"/>
+  </joint>
+  <!-- Left wheel back -->
+  <link name='left_wheel_back'>
+    <inertial>
+      <mass value="5.0"/>
+      <origin xyz="0.0 0 0" rpy=" 0 1.5707 1.5707"/>
+      <inertia
+          ixx="0.1" ixy="0" ixz="0"
+          iyy="0.1" iyz="0"
+          izz="0.1"
+      />
+    </inertial>
+    <collision name='left_wheel_back_collision'>
+      <origin xyz="0 0 0" rpy=" 0 1.5707 1.5707"/>
+      <geometry>
+        <cylinder length="0.05" radius="0.1"/>
+      </geometry>
+    </collision>
+    <visual name='left_wheel_back_visual'>
+      <origin xyz="0 0 0" rpy=" 0 1.5705 1.5707"/>
+      <geometry>
+        <cylinder length="0.05" radius="0.1"/>
+      </geometry>
+    </visual>
+  </link>
+  <joint type="continuous" name="left_wheel_back_hinge">
+    <origin xyz="-0.15 0.15 0" rpy="0 0 0"/>
+    <child link="left_wheel_back"/>
+    <parent link="chassis"/>
+    <axis xyz="0 1 0" rpy="0 0 0"/>
+    <limit effort="10000" velocity="1000"/>
+    <dynamics damping="1.0" friction="1.0"/>
+  </joint>
+  <!-- Right wheel front -->
+  <link name='right_wheel_front'>
+    <inertial>
+      <mass value="5.0"/>
+      <origin xyz="0.0 0 0" rpy=" 0 1.5707 1.5707"/>
+      <inertia
+          ixx="0.1" ixy="0" ixz="0"
+          iyy="0.1" iyz="0"
+          izz="0.1"
+      />
+    </inertial>
+    <collision name='right_wheel_front_collision'>
+      <origin xyz="0 0 0" rpy=" 0 1.5707 1.5707"/>
+      <geometry>
+        <cylinder length="0.05" radius="0.1"/>
+      </geometry>
+    </collision>
+    <visual name='right_wheel_front_visual'>
+      <origin xyz="0 0 0" rpy=" 0 1.5705 1.5707"/>
+      <geometry>
+        <cylinder length="0.05" radius="0.1"/>
+      </geometry>
+    </visual>
+  </link>
+  <joint type="continuous" name="right_wheel_front_hinge">
+    <origin xyz="0.15 -0.15 0" rpy="0 0 0"/>
+    <child link="right_wheel_front"/>
+    <parent link="chassis"/>
+    <axis xyz="0 1 0" rpy="0 0 0"/>
+    <limit effort="10000" velocity="1000"/>
+    <dynamics damping="1.0" friction="1.0"/>
+  </joint>
+  <!-- Right wheel back -->
+  <link name='right_wheel_back'>
+    <inertial>
+      <mass value="5.0"/>
+      <origin xyz="0.0 0 0" rpy=" 0 1.5707 1.5707"/>
+      <inertia
+          ixx="0.1" ixy="0" ixz="0"
+          iyy="0.1" iyz="0"
+          izz="0.1"
+      />
+    </inertial>
+    <collision name='right_wheel_back_collision'>
+      <origin xyz="0 0 0" rpy=" 0 1.5707 1.5707"/>
+      <geometry>
+        <cylinder length="0.05" radius="0.1"/>
+      </geometry>
+    </collision>
+    <visual name='right_wheel_back_visual'>
+      <origin xyz="0 0 0" rpy=" 0 1.5705 1.5707"/>
+      <geometry>
+        <cylinder length="0.05" radius="0.1"/>
+      </geometry>
+    </visual>
+  </link>
+  <joint type="continuous" name="right_wheel_back_hinge">
+    <origin xyz="-0.15 -0.15 0" rpy="0 0 0"/>
+    <child link="right_wheel_back"/>
+    <parent link="chassis"/>
+    <axis xyz="0 1 0" rpy="0 0 0"/>
+    <limit effort="10000" velocity="1000"/>
+    <dynamics damping="1.0" friction="1.0"/>
+  </joint>
+  <!-- CAMERA -->
   <link name="camera">
     <inertial>
@@ -159,4 +209,5 @@
     <axis xyz="0 1 0" rpy="0 0 0"/>
   </joint>
+  <!-- LIDAR -->
   <link name="hokuyo">
     <inertial>
@@ -189,5 +240,5 @@
   </joint>
   <!-- IMU -->
-    <link name="imu_link">
+  <link name="imu_link">
     <inertial>
       <mass value="0.001"/>
@@ -209,5 +260,5 @@
   </link>
   <joint name="imu_joint" type="fixed">
-    <axis xyz="1 0 0"/> <!-- 0 1 0 -->
+    <axis xyz="1 0 0"/>
     <origin xyz="0 0 0.19"/>
     <parent link="chassis"/>

Commit message: add depth camera

File: urdf/robot.xacro (robot description, xacro)
@@ -179,8 +179,8 @@
     <dynamics damping="1.0" friction="1.0"/>
   </joint>
-  <!-- CAMERA -->
-  <link name="camera">
-    <inertial>
-      <mass value="0.1"/>
+  <!-- LIDAR -->
+  <link name="hokuyo">
+    <inertial>
+      <mass value="1e-5"/>
       <origin xyz="0 0 0" rpy=" 0 0 0"/>
       <inertia
@@ -190,34 +190,4 @@
       />
     </inertial>
-    <collision name='camera_collision'>
-      <origin xyz="0 0 0" rpy=" 0 0 0"/>
-      <geometry>
-        <box size="0.05 0.05 0.05"/>
-      </geometry>
-    </collision>
-    <visual name='camera_visual'>
-      <origin xyz="0 0 0" rpy=" 0 0 0"/>
-      <geometry>
-        <box size="0.05 0.05 0.05"/>
-      </geometry>
-    </visual>
-  </link>
-  <joint type="fixed" name="camera_joint">
-    <origin xyz="0.2 0 0" rpy="0 0 0"/>
-    <child link="camera"/>
-    <parent link="chassis"/>
-    <axis xyz="0 1 0" rpy="0 0 0"/>
-  </joint>
-  <!-- LIDAR -->
-  <link name="hokuyo">
-    <inertial>
-      <mass value="1e-5"/>
-      <origin xyz="0 0 0" rpy=" 0 0 0"/>
-      <inertia
-          ixx="1e-6" ixy="0" ixz="0"
-          iyy="1e-6" iyz="0"
-          izz="1e-6"
-      />
-    </inertial>
     <collision name='hokuyo_collision'>
       <origin xyz="0 0 0" rpy=" 0 0 0"/>
@@ -265,3 +235,9 @@
     <child link="imu_link"/>
   </joint>
+  <!-- Import macro for realsense-RS200 camera-->
+  <xacro:include filename="$(find gazebo_simulation)/urdf/realsense-RS200.macro.xacro"/>
+  <!-- Create camera instance -->
+  <xacro:realsense-rs200 prefix="" parent="chassis">
+    <origin xyz="0 0 .3" rpy="0 0 0" />
+  </xacro:realsense-rs200>
 </robot>

Commit message: camera is in front of the lidar

File: urdf/robot.xacro (robot description, xacro)
@@ -239,5 +239,5 @@
   <!-- Create camera instance -->
   <xacro:realsense-rs200 prefix="" parent="chassis">
-    <origin xyz="0 0 .3" rpy="0 0 0" />
+    <origin xyz="0.2 0 .07" rpy="0 0 0" />
   </xacro:realsense-rs200>
 </robot>

Commit message: Match robot dimentions to kuka youbot

File: urdf/robot.xacro (robot description, xacro)
@@ -3,8 +3,11 @@
 <xacro:include filename="$(find gazebo_simulation)/urdf/robot.gazebo" />
   <gazebo reference="chassis">
-    <material>Gazebo/White</material>
-  </gazebo>
-  <gazebo reference="camera">
-    <material>Gazebo/Grey</material>
+    <material>Gazebo/RedBright</material>
+  </gazebo>
+  <gazebo reference="chassis2">
+    <material>Gazebo/RedBright</material>
+  </gazebo>
+  <gazebo reference="robot_lidar_platform">
+    <material>Gazebo/RedBright</material>
   </gazebo>
   <gazebo reference="left_wheel_front">
@@ -22,4 +25,8 @@
   <!-- ROBOT description -->
   <link name="robot_footprint"></link>
+  <!--
+    KUKA youBot dimentions
+    https://www.expo21xx.com/industrial-robots/20317_st3_mobile-robot-research/default.htm
+  -->
   <joint name="robot_footprint_joint" type="fixed">
     <origin xyz="0 0 0" rpy="0 0 0" />
@@ -41,5 +48,5 @@
       <origin xyz="0 0 0" rpy=" 0 0 0"/>
       <geometry>
-        <box size=".4 .2 .1"/>
+        <box size=".580 .210 .110"/>
       </geometry>
     </collision>
@@ -47,12 +54,74 @@
       <origin xyz="0 0 0" rpy=" 0 0 0"/>
       <geometry>
-        <box size=".4 .2 .1"/>
-      </geometry>
-    </visual>
-  </link>
+        <box size=".580 .210 .110"/>
+      </geometry>
+    </visual>
+  </link>
+  <joint name="robot_footprint_joint2" type="fixed">
+    <origin xyz="0 0 0" rpy="0 0 0" />
+    <parent link="robot_footprint"/>
+    <child link="chassis2" />
+  </joint>
+  <link name='chassis2'>
+    <inertial>
+      <mass value="1.0"/>
+      <origin xyz="0.0 0 0" rpy=" 0 0 0"/>
+      <inertia
+          ixx="0.1" ixy="0" ixz="0"
+          iyy="0.1" iyz="0"
+          izz="0.1"
+      />
+    </inertial>
+    <collision name='collision2'>
+      <origin xyz="0 0 0" rpy=" 0 0 0"/>
+      <geometry>
+        <box size=".370 .380 .110"/>
+      </geometry>
+    </collision>
+    <visual name='chassis2_visual'>
+      <origin xyz="0 0 0" rpy=" 0 0 0"/>
+      <geometry>
+        <box size=".370 .380 .110"/>
+      </geometry>
+    </visual>
+  </link>
+  <joint name="robot_lidar_platform_joint" type="fixed">
+    <origin xyz="0.32 0 -0.05" rpy="0 0 0" />
+    <parent link="robot_footprint"/>
+    <child link="robot_lidar_platform" />
+  </joint>
+  <link name='robot_lidar_platform'>
+    <inertial>
+      <mass value="1.0"/>
+      <origin xyz="0.0 0 0" rpy=" 0 0 0"/>
+      <inertia
+          ixx="0.1" ixy="0" ixz="0"
+          iyy="0.1" iyz="0"
+          izz="0.1"
+      />
+    </inertial>
+    <collision name='collision2'>
+      <origin xyz="0 0 0" rpy=" 0 0 0"/>
+      <geometry>
+        <box size=".12 .10 .01"/>
+      </geometry>
+    </collision>
+    <visual name='chassis2_visual'>
+      <origin xyz="0.0 0 0" rpy=" 0 0 0"/>
+      <geometry>
+        <box size=".12 .10 .01"/>
+      </geometry>
+    </visual>
+  </link>
+  <!--
+  Wheel:
+    radius: 50mm
+    length: 76mm
+    mass: 500gr.
+  -->
   <!-- Left wheel front -->
   <link name='left_wheel_front'>
     <inertial>
-      <mass value="5.0"/>
+      <mass value="0.5"/>
       <origin xyz="0.0 0 0" rpy=" 0 1.5707 1.5707"/>
       <inertia
@@ -65,5 +134,5 @@
       <origin xyz="0 0 0" rpy=" 0 1.5707 1.5707"/>
       <geometry>
-        <cylinder length="0.05" radius="0.1"/>
+        <cylinder length="0.076" radius="0.05"/>
       </geometry>
     </collision>
@@ -71,10 +140,10 @@
       <origin xyz="0 0 0" rpy=" 0 1.5705 1.5707"/>
       <geometry>
-        <cylinder length="0.05" radius="0.1"/>
+        <cylinder length="0.076" radius="0.05"/>
       </geometry>
     </visual>
   </link>
   <joint type="continuous" name="left_wheel_front_hinge">
-    <origin xyz="0.15 0.15 0" rpy="0 0 0"/>
+    <origin xyz="0.25 0.15 -0.03" rpy="0 0 0"/>
     <child link="left_wheel_front"/>
     <parent link="chassis"/>
@@ -86,5 +155,5 @@
   <link name='left_wheel_back'>
     <inertial>
-      <mass value="5.0"/>
+      <mass value="0.5"/>
       <origin xyz="0.0 0 0" rpy=" 0 1.5707 1.5707"/>
       <inertia
@@ -97,5 +166,5 @@
       <origin xyz="0 0 0" rpy=" 0 1.5707 1.5707"/>
       <geometry>
-        <cylinder length="0.05" radius="0.1"/>
+        <cylinder length="0.076" radius="0.05"/>
       </geometry>
     </collision>
@@ -103,10 +172,10 @@
       <origin xyz="0 0 0" rpy=" 0 1.5705 1.5707"/>
       <geometry>
-        <cylinder length="0.05" radius="0.1"/>
+        <cylinder length="0.076" radius="0.05"/>
       </geometry>
     </visual>
   </link>
   <joint type="continuous" name="left_wheel_back_hinge">
-    <origin xyz="-0.15 0.15 0" rpy="0 0 0"/>
+    <origin xyz="-0.25 0.15 -0.03" rpy="0 0 0"/>
     <child link="left_wheel_back"/>
     <parent link="chassis"/>
@@ -118,5 +187,5 @@
   <link name='right_wheel_front'>
     <inertial>
-      <mass value="5.0"/>
+      <mass value="0.5"/>
       <origin xyz="0.0 0 0" rpy=" 0 1.5707 1.5707"/>
       <inertia
@@ -129,5 +198,5 @@
       <origin xyz="0 0 0" rpy=" 0 1.5707 1.5707"/>
       <geometry>
-        <cylinder length="0.05" radius="0.1"/>
+        <cylinder length="0.076" radius="0.05"/>
       </geometry>
     </collision>
@@ -135,10 +204,10 @@
       <origin xyz="0 0 0" rpy=" 0 1.5705 1.5707"/>
       <geometry>
-        <cylinder length="0.05" radius="0.1"/>
+        <cylinder length="0.076" radius="0.05"/>
       </geometry>
     </visual>
   </link>
   <joint type="continuous" name="right_wheel_front_hinge">
-    <origin xyz="0.15 -0.15 0" rpy="0 0 0"/>
+    <origin xyz="0.25 -0.15 -0.03" rpy="0 0 0"/>
     <child link="right_wheel_front"/>
     <parent link="chassis"/>
@@ -150,5 +219,5 @@
   <link name='right_wheel_back'>
     <inertial>
-      <mass value="5.0"/>
+      <mass value="0.5"/>
       <origin xyz="0.0 0 0" rpy=" 0 1.5707 1.5707"/>
       <inertia
@@ -161,5 +230,5 @@
       <origin xyz="0 0 0" rpy=" 0 1.5707 1.5707"/>
       <geometry>
-        <cylinder length="0.05" radius="0.1"/>
+        <cylinder length="0.076" radius="0.05"/>
       </geometry>
     </collision>
@@ -167,10 +236,10 @@
       <origin xyz="0 0 0" rpy=" 0 1.5705 1.5707"/>
       <geometry>
-        <cylinder length="0.05" radius="0.1"/>
+        <cylinder length="0.076" radius="0.05"/>
       </geometry>
     </visual>
   </link>
   <joint type="continuous" name="right_wheel_back_hinge">
-    <origin xyz="-0.15 -0.15 0" rpy="0 0 0"/>
+    <origin xyz="-0.25 -0.15 -0.03" rpy="0 0 0"/>
     <child link="right_wheel_back"/>
     <parent link="chassis"/>
@@ -204,5 +273,5 @@
   </link>
   <joint type="fixed" name="hokuyo_joint">
-    <origin xyz="0.15 0 0.1" rpy="0 0 0"/>
+    <origin xyz="0.34 0 -0.0099" rpy="0 0 0"/>
     <child link="hokuyo"/>
     <parent link="chassis"/>
@@ -239,5 +308,5 @@
   <!-- Create camera instance -->
   <xacro:realsense-rs200 prefix="" parent="chassis">
-    <origin xyz="0.2 0 .07" rpy="0 0 0" />
+    <origin xyz="0.285 0 .065" rpy="0 0 0" />
   </xacro:realsense-rs200>
 </robot>
