Commit message: Revert "Match robot dimentions to kuka youbot"
This reverts commit d19f0842faf7728c9f81d49af749ab6debf67136.

File: urdf/robot.xacro (robot description, xacro)
@@ -3,11 +3,8 @@
 <xacro:include filename="$(find gazebo_simulation)/urdf/robot.gazebo" />
   <gazebo reference="chassis">
-    <material>Gazebo/RedBright</material>
-  </gazebo>
-  <gazebo reference="chassis2">
-    <material>Gazebo/RedBright</material>
-  </gazebo>
-  <gazebo reference="robot_lidar_platform">
-    <material>Gazebo/RedBright</material>
+    <material>Gazebo/White</material>
+  </gazebo>
+  <gazebo reference="camera">
+    <material>Gazebo/Grey</material>
   </gazebo>
   <gazebo reference="left_wheel_front">
@@ -25,8 +22,4 @@
   <!-- ROBOT description -->
   <link name="robot_footprint"></link>
-  <!--
-    KUKA youBot dimentions
-    https://www.expo21xx.com/industrial-robots/20317_st3_mobile-robot-research/default.htm
-  -->
   <joint name="robot_footprint_joint" type="fixed">
     <origin xyz="0 0 0" rpy="0 0 0" />
@@ -48,5 +41,5 @@
       <origin xyz="0 0 0" rpy=" 0 0 0"/>
       <geometry>
-        <box size=".580 .210 .110"/>
+        <box size=".4 .2 .1"/>
       </geometry>
     </collision>
@@ -54,74 +47,12 @@
       <origin xyz="0 0 0" rpy=" 0 0 0"/>
       <geometry>
-        <box size=".580 .210 .110"/>
-      </geometry>
-    </visual>
-  </link>
-  <joint name="robot_footprint_joint2" type="fixed">
-    <origin xyz="0 0 0" rpy="0 0 0" />
-    <parent link="robot_footprint"/>
-    <child link="chassis2" />
-  </joint>
-  <link name='chassis2'>
-    <inertial>
-      <mass value="1.0"/>
-      <origin xyz="0.0 0 0" rpy=" 0 0 0"/>
-      <inertia
-          ixx="0.1" ixy="0" ixz="0"
-          iyy="0.1" iyz="0"
-          izz="0.1"
-      />
-    </inertial>
-    <collision name='collision2'>
-      <origin xyz="0 0 0" rpy=" 0 0 0"/>
-      <geometry>
-        <box size=".370 .380 .110"/>
-      </geometry>
-    </collision>
-    <visual name='chassis2_visual'>
-      <origin xyz="0 0 0" rpy=" 0 0 0"/>
-      <geometry>
-        <box size=".370 .380 .110"/>
-      </geometry>
-    </visual>
-  </link>
-  <joint name="robot_lidar_platform_joint" type="fixed">
-    <origin xyz="0.32 0 -0.05" rpy="0 0 0" />
-    <parent link="robot_footprint"/>
-    <child link="robot_lidar_platform" />
-  </joint>
-  <link name='robot_lidar_platform'>
-    <inertial>
-      <mass value="1.0"/>
-      <origin xyz="0.0 0 0" rpy=" 0 0 0"/>
-      <inertia
-          ixx="0.1" ixy="0" ixz="0"
-          iyy="0.1" iyz="0"
-          izz="0.1"
-      />
-    </inertial>
-    <collision name='collision2'>
-      <origin xyz="0 0 0" rpy=" 0 0 0"/>
-      <geometry>
-        <box size=".12 .10 .01"/>
-      </geometry>
-    </collision>
-    <visual name='chassis2_visual'>
-      <origin xyz="0.0 0 0" rpy=" 0 0 0"/>
-      <geometry>
-        <box size=".12 .10 .01"/>
-      </geometry>
-    </visual>
-  </link>
-  <!--
-  Wheel:
-    radius: 50mm
-    length: 76mm
-    mass: 500gr.
-  -->
+        <box size=".4 .2 .1"/>
+      </geometry>
+    </visual>
+  </link>
   <!-- Left wheel front -->
   <link name='left_wheel_front'>
     <inertial>
-      <mass value="0.5"/>
+      <mass value="5.0"/>
       <origin xyz="0.0 0 0" rpy=" 0 1.5707 1.5707"/>
       <inertia
@@ -134,5 +65,5 @@
       <origin xyz="0 0 0" rpy=" 0 1.5707 1.5707"/>
       <geometry>
-        <cylinder length="0.076" radius="0.05"/>
+        <cylinder length="0.05" radius="0.1"/>
       </geometry>
     </collision>
@@ -140,10 +71,10 @@
       <origin xyz="0 0 0" rpy=" 0 1.5705 1.5707"/>
       <geometry>
-        <cylinder length="0.076" radius="0.05"/>
+        <cylinder length="0.05" radius="0.1"/>
       </geometry>
     </visual>
   </link>
   <joint type="continuous" name="left_wheel_front_hinge">
-    <origin xyz="0.25 0.15 -0.03" rpy="0 0 0"/>
+    <origin xyz="0.15 0.15 0" rpy="0 0 0"/>
     <child link="left_wheel_front"/>
     <parent link="chassis"/>
@@ -155,5 +86,5 @@
   <link name='left_wheel_back'>
     <inertial>
-      <mass value="0.5"/>
+      <mass value="5.0"/>
       <origin xyz="0.0 0 0" rpy=" 0 1.5707 1.5707"/>
       <inertia
@@ -166,5 +97,5 @@
       <origin xyz="0 0 0" rpy=" 0 1.5707 1.5707"/>
       <geometry>
-        <cylinder length="0.076" radius="0.05"/>
+        <cylinder length="0.05" radius="0.1"/>
       </geometry>
     </collision>
@@ -172,10 +103,10 @@
       <origin xyz="0 0 0" rpy=" 0 1.5705 1.5707"/>
       <geometry>
-        <cylinder length="0.076" radius="0.05"/>
+        <cylinder length="0.05" radius="0.1"/>
       </geometry>
     </visual>
   </link>
   <joint type="continuous" name="left_wheel_back_hinge">
-    <origin xyz="-0.25 0.15 -0.03" rpy="0 0 0"/>
+    <origin xyz="-0.15 0.15 0" rpy="0 0 0"/>
     <child link="left_wheel_back"/>
     <parent link="chassis"/>
@@ -187,5 +118,5 @@
   <link name='right_wheel_front'>
     <inertial>
-      <mass value="0.5"/>
+      <mass value="5.0"/>
       <origin xyz="0.0 0 0" rpy=" 0 1.5707 1.5707"/>
       <inertia
@@ -198,5 +129,5 @@
       <origin xyz="0 0 0" rpy=" 0 1.5707 1.5707"/>
       <geometry>
-        <cylinder length="0.076" radius="0.05"/>
+        <cylinder length="0.05" radius="0.1"/>
       </geometry>
     </collision>
@@ -204,10 +135,10 @@
       <origin xyz="0 0 0" rpy=" 0 1.5705 1.5707"/>
       <geometry>
-        <cylinder length="0.076" radius="0.05"/>
+        <cylinder length="0.05" radius="0.1"/>
       </geometry>
     </visual>
   </link>
   <joint type="continuous" name="right_wheel_front_hinge">
-    <origin xyz="0.25 -0.15 -0.03" rpy="0 0 0"/>
+    <origin xyz="0.15 -0.15 0" rpy="0 0 0"/>
     <child link="right_wheel_front"/>
     <parent link="chassis"/>
@@ -219,5 +150,5 @@
   <link name='right_wheel_back'>
     <inertial>
-      <mass value="0.5"/>
+      <mass value="5.0"/>
       <origin xyz="0.0 0 0" rpy=" 0 1.5707 1.5707"/>
       <inertia
@@ -230,5 +161,5 @@
       <origin xyz="0 0 0" rpy=" 0 1.5707 1.5707"/>
       <geometry>
-        <cylinder length="0.076" radius="0.05"/>
+        <cylinder length="0.05" radius="0.1"/>
       </geometry>
     </collision>
@@ -236,10 +167,10 @@
       <origin xyz="0 0 0" rpy=" 0 1.5705 1.5707"/>
       <geometry>
-        <cylinder length="0.076" radius="0.05"/>
+        <cylinder length="0.05" radius="0.1"/>
       </geometry>
     </visual>
   </link>
   <joint type="continuous" name="right_wheel_back_hinge">
-    <origin xyz="-0.25 -0.15 -0.03" rpy="0 0 0"/>
+    <origin xyz="-0.15 -0.15 0" rpy="0 0 0"/>
     <child link="right_wheel_back"/>
     <parent link="chassis"/>
@@ -273,5 +204,5 @@
   </link>
   <joint type="fixed" name="hokuyo_joint">
-    <origin xyz="0.34 0 -0.0099" rpy="0 0 0"/>
+    <origin xyz="0.15 0 0.1" rpy="0 0 0"/>
     <child link="hokuyo"/>
     <parent link="chassis"/>
@@ -308,5 +239,5 @@
   <!-- Create camera instance -->
   <xacro:realsense-rs200 prefix="" parent="chassis">
-    <origin xyz="0.285 0 .065" rpy="0 0 0" />
+    <origin xyz="0.2 0 .07" rpy="0 0 0" />
   </xacro:realsense-rs200>
 </robot>

Commit message: new definition of the robot close to dims of kuka youbot

File: urdf/robot.xacro (robot description, xacro)
@@ -3,8 +3,11 @@
 <xacro:include filename="$(find gazebo_simulation)/urdf/robot.gazebo" />
   <gazebo reference="chassis">
-    <material>Gazebo/White</material>
-  </gazebo>
-  <gazebo reference="camera">
-    <material>Gazebo/Grey</material>
+    <material>Gazebo/RedBright</material>
+  </gazebo>
+  <gazebo reference="chassis2">
+    <material>Gazebo/RedBright</material>
+  </gazebo>
+  <gazebo reference="robot_lidar_platform">
+    <material>Gazebo/RedBright</material>
   </gazebo>
   <gazebo reference="left_wheel_front">
@@ -22,4 +25,8 @@
   <!-- ROBOT description -->
   <link name="robot_footprint"></link>
+  <!--
+    KUKA youBot dimentions
+    https://www.expo21xx.com/industrial-robots/20317_st3_mobile-robot-research/default.htm
+  -->
   <joint name="robot_footprint_joint" type="fixed">
     <origin xyz="0 0 0" rpy="0 0 0" />
@@ -41,5 +48,5 @@
       <origin xyz="0 0 0" rpy=" 0 0 0"/>
       <geometry>
-        <box size=".4 .2 .1"/>
+        <box size=".580 .210 .110"/>
       </geometry>
     </collision>
@@ -47,12 +54,74 @@
       <origin xyz="0 0 0" rpy=" 0 0 0"/>
       <geometry>
-        <box size=".4 .2 .1"/>
-      </geometry>
-    </visual>
-  </link>
+        <box size=".580 .210 .110"/>
+      </geometry>
+    </visual>
+  </link>
+  <joint name="robot_footprint_joint2" type="fixed">
+    <origin xyz="0 0 0" rpy="0 0 0" />
+    <parent link="chassis"/>
+    <child link="chassis2" />
+  </joint>
+  <link name='chassis2'>
+    <inertial>
+      <mass value="1.0"/>
+      <origin xyz="0.0 0 0" rpy=" 0 0 0"/>
+      <inertia
+          ixx="0.1" ixy="0" ixz="0"
+          iyy="0.1" iyz="0"
+          izz="0.1"
+      />
+    </inertial>
+    <collision name='collision2'>
+      <origin xyz="0 0 0" rpy=" 0 0 0"/>
+      <geometry>
+        <box size=".370 .380 .110"/>
+      </geometry>
+    </collision>
+    <visual name='chassis2_visual'>
+      <origin xyz="0 0 0" rpy=" 0 0 0"/>
+      <geometry>
+        <box size=".370 .380 .110"/>
+      </geometry>
+    </visual>
+  </link>
+  <joint name="robot_lidar_platform_joint" type="fixed">
+    <origin xyz="0.32 0 -0.05" rpy="0 0 0" />
+    <parent link="chassis"/>
+    <child link="robot_lidar_platform" />
+  </joint>
+  <link name='robot_lidar_platform'>
+    <inertial>
+      <mass value="1.0"/>
+      <origin xyz="0.0 0 0" rpy=" 0 0 0"/>
+      <inertia
+          ixx="0.1" ixy="0" ixz="0"
+          iyy="0.1" iyz="0"
+          izz="0.1"
+      />
+    </inertial>
+    <collision name='collision2'>
+      <origin xyz="0 0 0" rpy=" 0 0 0"/>
+      <geometry>
+        <box size=".12 .10 .01"/>
+      </geometry>
+    </collision>
+    <visual name='chassis2_visual'>
+      <origin xyz="0.0 0 0" rpy=" 0 0 0"/>
+      <geometry>
+        <box size=".12 .10 .01"/>
+      </geometry>
+    </visual>
+  </link>
+  <!--
+  Wheel:
+    radius: 50mm
+    length: 76mm
+    mass: 500gr.
+  -->
   <!-- Left wheel front -->
   <link name='left_wheel_front'>
     <inertial>
-      <mass value="5.0"/>
+      <mass value="0.5"/>
       <origin xyz="0.0 0 0" rpy=" 0 1.5707 1.5707"/>
       <inertia
@@ -65,5 +134,5 @@
       <origin xyz="0 0 0" rpy=" 0 1.5707 1.5707"/>
       <geometry>
-        <cylinder length="0.05" radius="0.1"/>
+        <cylinder length="0.076" radius="0.05"/>
       </geometry>
     </collision>
@@ -71,10 +140,10 @@
       <origin xyz="0 0 0" rpy=" 0 1.5705 1.5707"/>
       <geometry>
-        <cylinder length="0.05" radius="0.1"/>
+        <cylinder length="0.076" radius="0.05"/>
       </geometry>
     </visual>
   </link>
   <joint type="continuous" name="left_wheel_front_hinge">
-    <origin xyz="0.15 0.15 0" rpy="0 0 0"/>
+    <origin xyz="0.25 0.15 -0.03" rpy="0 0 0"/>
     <child link="left_wheel_front"/>
     <parent link="chassis"/>
@@ -86,5 +155,5 @@
   <link name='left_wheel_back'>
     <inertial>
-      <mass value="5.0"/>
+      <mass value="0.5"/>
       <origin xyz="0.0 0 0" rpy=" 0 1.5707 1.5707"/>
       <inertia
@@ -97,5 +166,5 @@
       <origin xyz="0 0 0" rpy=" 0 1.5707 1.5707"/>
       <geometry>
-        <cylinder length="0.05" radius="0.1"/>
+        <cylinder length="0.076" radius="0.05"/>
       </geometry>
     </collision>
@@ -103,10 +172,10 @@
       <origin xyz="0 0 0" rpy=" 0 1.5705 1.5707"/>
       <geometry>
-        <cylinder length="0.05" radius="0.1"/>
+        <cylinder length="0.076" radius="0.05"/>
       </geometry>
     </visual>
   </link>
   <joint type="continuous" name="left_wheel_back_hinge">
-    <origin xyz="-0.15 0.15 0" rpy="0 0 0"/>
+    <origin xyz="-0.25 0.15 -0.03" rpy="0 0 0"/>
     <child link="left_wheel_back"/>
     <parent link="chassis"/>
@@ -118,5 +187,5 @@
   <link name='right_wheel_front'>
     <inertial>
-      <mass value="5.0"/>
+      <mass value="0.5"/>
       <origin xyz="0.0 0 0" rpy=" 0 1.5707 1.5707"/>
       <inertia
@@ -129,5 +198,5 @@
       <origin xyz="0 0 0" rpy=" 0 1.5707 1.5707"/>
       <geometry>
-        <cylinder length="0.05" radius="0.1"/>
+        <cylinder length="0.076" radius="0.05"/>
       </geometry>
     </collision>
@@ -135,10 +204,10 @@
       <origin xyz="0 0 0" rpy=" 0 1.5705 1.5707"/>
       <geometry>
-        <cylinder length="0.05" radius="0.1"/>
+        <cylinder length="0.076" radius="0.05"/>
       </geometry>
     </visual>
   </link>
   <joint type="continuous" name="right_wheel_front_hinge">
-    <origin xyz="0.15 -0.15 0" rpy="0 0 0"/>
+    <origin xyz="0.25 -0.15 -0.03" rpy="0 0 0"/>
     <child link="right_wheel_front"/>
     <parent link="chassis"/>
@@ -150,5 +219,5 @@
   <link name='right_wheel_back'>
     <inertial>
-      <mass value="5.0"/>
+      <mass value="0.5"/>
       <origin xyz="0.0 0 0" rpy=" 0 1.5707 1.5707"/>
       <inertia
@@ -161,5 +230,5 @@
       <origin xyz="0 0 0" rpy=" 0 1.5707 1.5707"/>
       <geometry>
-        <cylinder length="0.05" radius="0.1"/>
+        <cylinder length="0.076" radius="0.05"/>
       </geometry>
     </collision>
@@ -167,10 +236,10 @@
       <origin xyz="0 0 0" rpy=" 0 1.5705 1.5707"/>
       <geometry>
-        <cylinder length="0.05" radius="0.1"/>
+        <cylinder length="0.076" radius="0.05"/>
       </geometry>
     </visual>
   </link>
   <joint type="continuous" name="right_wheel_back_hinge">
-    <origin xyz="-0.15 -0.15 0" rpy="0 0 0"/>
+    <origin xyz="-0.25 -0.15 -0.03" rpy="0 0 0"/>
     <child link="right_wheel_back"/>
     <parent link="chassis"/>
@@ -204,5 +273,5 @@
   </link>
   <joint type="fixed" name="hokuyo_joint">
-    <origin xyz="0.15 0 0.1" rpy="0 0 0"/>
+    <origin xyz="0.34 0 -0.0099" rpy="0 0 0"/>
     <child link="hokuyo"/>
     <parent link="chassis"/>
@@ -239,5 +308,5 @@
   <!-- Create camera instance -->
   <xacro:realsense-rs200 prefix="" parent="chassis">
-    <origin xyz="0.2 0 .07" rpy="0 0 0" />
+    <origin xyz="0.285 0 .065" rpy="0 0 0" />
   </xacro:realsense-rs200>
 </robot>

Commit message: wooden wheels

File: urdf/robot.xacro (robot description, xacro)
@@ -12,14 +12,14 @@
   </gazebo>
   <gazebo reference="left_wheel_front">
-    <material>Gazebo/Black</material>
+    <material>Gazebo/Wood</material>
   </gazebo>
   <gazebo reference="right_wheel_front">
-    <material>Gazebo/Black</material>
+    <material>Gazebo/Wood</material>
   </gazebo>
   <gazebo reference="left_wheel_back">
-    <material>Gazebo/Black</material>
+    <material>Gazebo/Wood</material>
   </gazebo>
   <gazebo reference="right_wheel_back">
-    <material>Gazebo/Black</material>
+    <material>Gazebo/Wood</material>
   </gazebo>
   <!-- ROBOT description -->

Commit message: check all driving modes

File: urdf/robot.xacro (robot description, xacro)
@@ -48,5 +48,5 @@
       <origin xyz="0 0 0" rpy=" 0 0 0"/>
       <geometry>
-        <box size=".580 .210 .110"/>
+        <box size=".580 .270 .110"/>
       </geometry>
     </collision>
@@ -54,5 +54,5 @@
       <origin xyz="0 0 0" rpy=" 0 0 0"/>
       <geometry>
-        <box size=".580 .210 .110"/>
+        <box size=".580 .270 .110"/>
       </geometry>
     </visual>
@@ -76,5 +76,5 @@
       <origin xyz="0 0 0" rpy=" 0 0 0"/>
       <geometry>
-        <box size=".370 .380 .110"/>
+        <box size=".280 .400 .110"/>
       </geometry>
     </collision>
@@ -82,5 +82,5 @@
       <origin xyz="0 0 0" rpy=" 0 0 0"/>
       <geometry>
-        <box size=".370 .380 .110"/>
+        <box size=".280 .400 .110"/>
       </geometry>
     </visual>
@@ -134,5 +134,5 @@
       <origin xyz="0 0 0" rpy=" 0 1.5707 1.5707"/>
       <geometry>
-        <cylinder length="0.076" radius="0.05"/>
+        <cylinder length="0.07" radius="0.05"/>
       </geometry>
     </collision>
@@ -140,10 +140,10 @@
       <origin xyz="0 0 0" rpy=" 0 1.5705 1.5707"/>
       <geometry>
-        <cylinder length="0.076" radius="0.05"/>
+        <cylinder length="0.07" radius="0.05"/>
       </geometry>
     </visual>
   </link>
   <joint type="continuous" name="left_wheel_front_hinge">
-    <origin xyz="0.25 0.15 -0.03" rpy="0 0 0"/>
+    <origin xyz="0.2 0.18 -0.03" rpy="0 0 0"/>
     <child link="left_wheel_front"/>
     <parent link="chassis"/>
@@ -166,5 +166,5 @@
       <origin xyz="0 0 0" rpy=" 0 1.5707 1.5707"/>
       <geometry>
-        <cylinder length="0.076" radius="0.05"/>
+        <cylinder length="0.07" radius="0.05"/>
       </geometry>
     </collision>
@@ -172,10 +172,10 @@
       <origin xyz="0 0 0" rpy=" 0 1.5705 1.5707"/>
       <geometry>
-        <cylinder length="0.076" radius="0.05"/>
+        <cylinder length="0.07" radius="0.05"/>
       </geometry>
     </visual>
   </link>
   <joint type="continuous" name="left_wheel_back_hinge">
-    <origin xyz="-0.25 0.15 -0.03" rpy="0 0 0"/>
+    <origin xyz="-0.2 0.18 -0.03" rpy="0 0 0"/>
     <child link="left_wheel_back"/>
     <parent link="chassis"/>
@@ -198,5 +198,5 @@
       <origin xyz="0 0 0" rpy=" 0 1.5707 1.5707"/>
       <geometry>
-        <cylinder length="0.076" radius="0.05"/>
+        <cylinder length="0.07" radius="0.05"/>
       </geometry>
     </collision>
@@ -204,10 +204,10 @@
       <origin xyz="0 0 0" rpy=" 0 1.5705 1.5707"/>
       <geometry>
-        <cylinder length="0.076" radius="0.05"/>
+        <cylinder length="0.07" radius="0.05"/>
       </geometry>
     </visual>
   </link>
   <joint type="continuous" name="right_wheel_front_hinge">
-    <origin xyz="0.25 -0.15 -0.03" rpy="0 0 0"/>
+    <origin xyz="0.2 -0.18 -0.03" rpy="0 0 0"/>
     <child link="right_wheel_front"/>
     <parent link="chassis"/>
@@ -230,5 +230,5 @@
       <origin xyz="0 0 0" rpy=" 0 1.5707 1.5707"/>
       <geometry>
-        <cylinder length="0.076" radius="0.05"/>
+        <cylinder length="0.07" radius="0.05"/>
       </geometry>
     </collision>
@@ -236,10 +236,10 @@
       <origin xyz="0 0 0" rpy=" 0 1.5705 1.5707"/>
       <geometry>
-        <cylinder length="0.076" radius="0.05"/>
+        <cylinder length="0.07" radius="0.05"/>
       </geometry>
     </visual>
   </link>
   <joint type="continuous" name="right_wheel_back_hinge">
-    <origin xyz="-0.25 -0.15 -0.03" rpy="0 0 0"/>
+    <origin xyz="-0.2 -0.18 -0.03" rpy="0 0 0"/>
     <child link="right_wheel_back"/>
     <parent link="chassis"/>
