Commit message: Add omni wheels

File: urdf/robot.xacro (robot description, xacro)
@@ -2,4 +2,6 @@
 <robot name="robot" xmlns:xacro="http://www.ros.org/wiki/xacro">
 <xacro:include filename="$(find gazebo_simulation)/urdf/robot.gazebo" />
+<xacro:include filename="$(find gazebo_simulation)/urdf/realsense-RS200.macro.xacro"/>
+<xacro:include filename="$(find gazebo_simulation)/urdf/omni_wheel.urdf.xacro" />
   <gazebo reference="chassis">
     <material>Gazebo/RedBright</material>
@@ -10,16 +12,4 @@
   <gazebo reference="robot_lidar_platform">
     <material>Gazebo/RedBright</material>
-  </gazebo>
-  <gazebo reference="left_wheel_front">
-    <material>Gazebo/Black</material>
-  </gazebo>
-  <gazebo reference="right_wheel_front">
-    <material>Gazebo/Black</material>
-  </gazebo>
-  <gazebo reference="left_wheel_back">
-    <material>Gazebo/Black</material>
-  </gazebo>
-  <gazebo reference="right_wheel_back">
-    <material>Gazebo/Black</material>
   </gazebo>
   <!-- ROBOT description -->
@@ -76,5 +66,5 @@
       <origin xyz="0 0 0" rpy=" 0 0 0"/>
       <geometry>
-        <box size=".280 .400 .110"/>
+        <box size=".135 .400 .110"/>
       </geometry>
     </collision>
@@ -82,5 +72,5 @@
       <origin xyz="0 0 0" rpy=" 0 0 0"/>
       <geometry>
-        <box size=".280 .400 .110"/>
+        <box size=".135 .400 .110"/>
       </geometry>
     </visual>
@@ -120,132 +110,4 @@
     mass: 500gr.
   -->
-  <!-- Left wheel front -->
-  <link name='left_wheel_front'>
-    <inertial>
-      <mass value="0.5"/>
-      <origin xyz="0.0 0 0" rpy=" 0 1.5707 1.5707"/>
-      <inertia
-          ixx="0.1" ixy="0" ixz="0"
-          iyy="0.1" iyz="0"
-          izz="0.1"
-      />
-    </inertial>
-    <collision name='left_wheel_front_collision'>
-      <origin xyz="0 0 0" rpy=" 0 1.5707 1.5707"/>
-      <geometry>
-        <cylinder length="0.07" radius="0.05"/>
-      </geometry>
-    </collision>
-    <visual name='left_wheel_front_visual'>
-      <origin xyz="0 0 0" rpy=" 0 1.5705 1.5707"/>
-      <geometry>
-        <cylinder length="0.07" radius="0.05"/>
-      </geometry>
-    </visual>
-  </link>
-  <joint type="continuous" name="left_wheel_front_hinge">
-    <origin xyz="0.2 0.18 -0.03" rpy="0 0 0"/>
-    <child link="left_wheel_front"/>
-    <parent link="chassis"/>
-    <axis xyz="0 1 0" rpy="0 0 0"/>
-    <limit effort="10000" velocity="1000"/>
-    <dynamics damping="1.0" friction="1.0"/>
-  </joint>
-  <!-- Left wheel back -->
-  <link name='left_wheel_back'>
-    <inertial>
-      <mass value="0.5"/>
-      <origin xyz="0.0 0 0" rpy=" 0 1.5707 1.5707"/>
-      <inertia
-          ixx="0.1" ixy="0" ixz="0"
-          iyy="0.1" iyz="0"
-          izz="0.1"
-      />
-    </inertial>
-    <collision name='left_wheel_back_collision'>
-      <origin xyz="0 0 0" rpy=" 0 1.5707 1.5707"/>
-      <geometry>
-        <cylinder length="0.07" radius="0.05"/>
-      </geometry>
-    </collision>
-    <visual name='left_wheel_back_visual'>
-      <origin xyz="0 0 0" rpy=" 0 1.5705 1.5707"/>
-      <geometry>
-        <cylinder length="0.07" radius="0.05"/>
-      </geometry>
-    </visual>
-  </link>
-  <joint type="continuous" name="left_wheel_back_hinge">
-    <origin xyz="-0.2 0.18 -0.03" rpy="0 0 0"/>
-    <child link="left_wheel_back"/>
-    <parent link="chassis"/>
-    <axis xyz="0 1 0" rpy="0 0 0"/>
-    <limit effort="10000" velocity="1000"/>
-    <dynamics damping="1.0" friction="1.0"/>
-  </joint>
-  <!-- Right wheel front -->
-  <link name='right_wheel_front'>
-    <inertial>
-      <mass value="0.5"/>
-      <origin xyz="0.0 0 0" rpy=" 0 1.5707 1.5707"/>
-      <inertia
-          ixx="0.1" ixy="0" ixz="0"
-          iyy="0.1" iyz="0"
-          izz="0.1"
-      />
-    </inertial>
-    <collision name='right_wheel_front_collision'>
-      <origin xyz="0 0 0" rpy=" 0 1.5707 1.5707"/>
-      <geometry>
-        <cylinder length="0.07" radius="0.05"/>
-      </geometry>
-    </collision>
-    <visual name='right_wheel_front_visual'>
-      <origin xyz="0 0 0" rpy=" 0 1.5705 1.5707"/>
-      <geometry>
-        <cylinder length="0.07" radius="0.05"/>
-      </geometry>
-    </visual>
-  </link>
-  <joint type="continuous" name="right_wheel_front_hinge">
-    <origin xyz="0.2 -0.18 -0.03" rpy="0 0 0"/>
-    <child link="right_wheel_front"/>
-    <parent link="chassis"/>
-    <axis xyz="0 1 0" rpy="0 0 0"/>
-    <limit effort="10000" velocity="1000"/>
-    <dynamics damping="1.0" friction="1.0"/>
-  </joint>
-  <!-- Right wheel back -->
-  <link name='right_wheel_back'>
-    <inertial>
-      <mass value="0.5"/>
-      <origin xyz="0.0 0 0" rpy=" 0 1.5707 1.5707"/>
-      <inertia
-          ixx="0.1" ixy="0" ixz="0"
-          iyy="0.1" iyz="0"
-          izz="0.1"
-      />
-    </inertial>
-    <collision name='right_wheel_back_collision'>
-      <origin xyz="0 0 0" rpy=" 0 1.5707 1.5707"/>
-      <geometry>
-        <cylinder length="0.07" radius="0.05"/>
-      </geometry>
-    </collision>
-    <visual name='right_wheel_back_visual'>
-      <origin xyz="0 0 0" rpy=" 0 1.5705 1.5707"/>
-      <geometry>
-        <cylinder length="0.07" radius="0.05"/>
-      </geometry>
-    </visual>
-  </link>
-  <joint type="continuous" name="right_wheel_back_hinge">
-    <origin xyz="-0.2 -0.18 -0.03" rpy="0 0 0"/>
-    <child link="right_wheel_back"/>
-    <parent link="chassis"/>
-    <axis xyz="0 1 0" rpy="0 0 0"/>
-    <limit effort="10000" velocity="1000"/>
-    <dynamics damping="1.0" friction="1.0"/>
-  </joint>
   <!-- LIDAR -->
   <link name="hokuyo">
@@ -304,9 +166,24 @@
     <child link="imu_link"/>
   </joint>
-  <!-- Import macro for realsense-RS200 camera-->
-  <xacro:include filename="$(find gazebo_simulation)/urdf/realsense-RS200.macro.xacro"/>
   <!-- Create camera instance -->
   <xacro:realsense-rs200 prefix="" parent="chassis">
     <origin xyz="0.285 0 .065" rpy="0 0 0" />
   </xacro:realsense-rs200>
+  <!-- x,y,z in translation from base_link to the center of the wheel -->
+  <xacro:property name="wheel_offset_x" value="0.2" />
+  <xacro:property name="wheel_offset_y" value="0.2" />
+  <xacro:property name="wheel_offset_z" value="0.0" />
+  <!-- Add omni wheels to the robot -->
+  <xacro:omni_wheel prefix="front_right" parent="chassis" reflect="false">
+    <origin xyz="${wheel_offset_x} -${wheel_offset_y} ${wheel_offset_z}" rpy="0 0 0"/>
+  </xacro:omni_wheel>
+  <xacro:omni_wheel prefix="front_left" parent="chassis" reflect="true">
+    <origin xyz="${wheel_offset_x} ${wheel_offset_y} ${wheel_offset_z}" rpy="0 0 0"/>
+  </xacro:omni_wheel>
+  <xacro:omni_wheel prefix="back_left" parent="chassis" reflect="true">
+    <origin xyz="-${wheel_offset_x} ${wheel_offset_y} ${wheel_offset_z}" rpy="0 0 0"/>
+  </xacro:omni_wheel>
+  <xacro:omni_wheel prefix="back_right" parent="chassis" reflect="false">
+    <origin xyz="-${wheel_offset_x} -${wheel_offset_y} ${wheel_offset_z}" rpy="0 0 0"/>
+  </xacro:omni_wheel>
 </robot>

Commit message: Put lidar position in the middle and on top

File: urdf/robot.xacro (robot description, xacro)
@@ -77,5 +77,5 @@
   </link>
   <joint name="robot_lidar_platform_joint" type="fixed">
-    <origin xyz="0.32 0 -0.05" rpy="0 0 0" />
+    <origin xyz="0.0 0.0 0.08" rpy="0 0 0" />
     <parent link="chassis"/>
     <child link="robot_lidar_platform" />
@@ -94,5 +94,5 @@
       <origin xyz="0 0 0" rpy=" 0 0 0"/>
       <geometry>
-        <box size=".12 .10 .01"/>
+        <box size=".12 .10 .10"/>
       </geometry>
     </collision>
@@ -100,5 +100,5 @@
       <origin xyz="0.0 0 0" rpy=" 0 0 0"/>
       <geometry>
-        <box size=".12 .10 .01"/>
+        <box size=".12 .10 .10"/>
       </geometry>
     </visual>
@@ -135,5 +135,5 @@
   </link>
   <joint type="fixed" name="hokuyo_joint">
-    <origin xyz="0.34 0 -0.0099" rpy="0 0 0"/>
+    <origin xyz="0.0 0.0 0.15" rpy="0 0 0"/>
     <child link="hokuyo"/>
     <parent link="chassis"/>

Commit message: switched to another IMU sensor (hector)
There were some range issues in cartographer_rosbag_validate:
W0424 23:07:41.895534 17317 rosbag_validate_main.cc:103] frame_id imu_link time 286544000000: IMU linear acceleration is 49.9795 m/s^2, expected is [3, 30] m/s^2. (It should include gravity and be given in m/s^2.) linear_acceleration 000049.011 -0.0895277 0009.79082

File: urdf/robot.xacro (robot description, xacro)
@@ -141,41 +141,26 @@
   </joint>
   <!-- IMU -->
+  <!-- from https://github.com/jackal/jackal/blob/indigo-devel/jackal_description/urdf/jackal.urdf.xacro -->
+  <xacro:property name="dummy_inertia" value="1e-09"/>
   <link name="imu_link">
     <inertial>
       <mass value="0.001"/>
-      <origin rpy="0 0 0" xyz="0 0 0"/>
-      <inertia ixx="0.0001" ixy="0" ixz="0" iyy="0.000001" iyz="0" izz="0.0001"/>
+      <origin xyz="0 0 0" rpy="0 0 0"/>
+      <inertia ixx="${dummy_inertia}" ixy="0.0" ixz="0.0" iyy="${dummy_inertia}" iyz="0.0" izz="${dummy_inertia}"/>
     </inertial>
-    <visual>
-      <origin rpy="0 0 0" xyz="0 0 0"/>
-      <geometry>
-        <box size="0.001 0.001 0.001"/>
-      </geometry>
-    </visual>
-    <collision>
-      <origin rpy="0 0 0" xyz="0 0 0"/>
-      <geometry>
-        <box size=".001 .001 .001"/>
-      </geometry>
-    </collision>
   </link>
-  <gazebo reference="imu_link">
-    <gravity>true</gravity>
-    <sensor name="imu_sensor" type="imu">
-      <always_on>true</always_on>
-      <update_rate>100</update_rate>
-      <visualize>true</visualize>
-      <topic>__default_topic__</topic>
-      <plugin filename="libgazebo_ros_imu_sensor.so" name="imu_plugin">
-        <topicName>imu</topicName>
-        <bodyName>imu_link</bodyName>
-        <updateRateHZ>10.0</updateRateHZ>
-        <gaussianNoise>0.0</gaussianNoise>
-        <xyzOffset>0 0 0</xyzOffset>
-        <rpyOffset>0 0 0</rpyOffset>
-        <frameName>imu_link</frameName>
-      </plugin>
-      <pose>0 0 0 0 0 0</pose>
-    </sensor>
+  <gazebo>
+    <plugin name="imu_controller" filename="libhector_gazebo_ros_imu.so">
+      <robotNamespace>/</robotNamespace>
+      <updateRate>50.0</updateRate>
+      <bodyName>imu_link</bodyName>
+      <topicName>imu</topicName>
+      <accelDrift>0.005 0.005 0.005</accelDrift>
+      <accelGaussianNoise>0.005 0.005 0.005</accelGaussianNoise>
+      <rateDrift>0.005 0.005 0.005 </rateDrift>
+      <rateGaussianNoise>0.005 0.005 0.005 </rateGaussianNoise>
+      <headingDrift>0.005</headingDrift>
+      <headingGaussianNoise>0.005</headingGaussianNoise>
+    </plugin>
   </gazebo>
   <joint name="imu_joint" type="fixed">

Commit message: cartographer seems working

File: urdf/robot.xacro (robot description, xacro)
@@ -4,8 +4,5 @@
 <xacro:include filename="$(find gazebo_simulation)/urdf/realsense-RS200.macro.xacro"/>
 <xacro:include filename="$(find gazebo_simulation)/urdf/omni_wheel.urdf.xacro" />
-  <gazebo reference="chassis">
-    <material>Gazebo/RedBright</material>
-  </gazebo>
-  <gazebo reference="chassis2">
+  <gazebo reference="base_link">
     <material>Gazebo/RedBright</material>
   </gazebo>
@@ -19,10 +16,5 @@
     https://www.expo21xx.com/industrial-robots/20317_st3_mobile-robot-research/default.htm
   -->
-  <joint name="robot_footprint_joint" type="fixed">
-    <origin xyz="0 0 0" rpy="0 0 0" />
-    <parent link="robot_footprint"/>
-    <child link="chassis" />
-  </joint>
-  <link name='chassis'>
+  <link name='base_link'>
     <pose>0 0 0.1 0 0 0</pose>
     <inertial>
@@ -41,5 +33,5 @@
       </geometry>
     </collision>
-    <visual name='chassis_visual'>
+    <visual name='base_link_visual'>
       <origin xyz="0 0 0" rpy=" 0 0 0"/>
       <geometry>
@@ -48,35 +40,12 @@
     </visual>
   </link>
-  <joint name="robot_footprint_joint2" type="fixed">
+  <joint name="robot_footprint_joint" type="fixed">
     <origin xyz="0 0 0" rpy="0 0 0" />
-    <parent link="chassis"/>
-    <child link="chassis2" />
+    <parent link="base_link" />
+    <child link="robot_footprint"/>
   </joint>
-  <link name='chassis2'>
-    <inertial>
-      <mass value="1.0"/>
-      <origin xyz="0.0 0 0" rpy=" 0 0 0"/>
-      <inertia
-          ixx="0.1" ixy="0" ixz="0"
-          iyy="0.1" iyz="0"
-          izz="0.1"
-      />
-    </inertial>
-    <collision name='collision2'>
-      <origin xyz="0 0 0" rpy=" 0 0 0"/>
-      <geometry>
-        <box size=".135 .400 .110"/>
-      </geometry>
-    </collision>
-    <visual name='chassis2_visual'>
-      <origin xyz="0 0 0" rpy=" 0 0 0"/>
-      <geometry>
-        <box size=".135 .400 .110"/>
-      </geometry>
-    </visual>
-  </link>
   <joint name="robot_lidar_platform_joint" type="fixed">
     <origin xyz="0.0 0.0 0.08" rpy="0 0 0" />
-    <parent link="chassis"/>
+    <parent link="base_link"/>
     <child link="robot_lidar_platform" />
   </joint>
@@ -97,5 +66,5 @@
       </geometry>
     </collision>
-    <visual name='chassis2_visual'>
+    <visual>
       <origin xyz="0.0 0 0" rpy=" 0 0 0"/>
       <geometry>
@@ -137,5 +106,5 @@
     <origin xyz="0.0 0.0 0.15" rpy="0 0 0"/>
     <child link="hokuyo"/>
-    <parent link="chassis"/>
+    <parent link="base_link"/>
     <axis xyz="0 1 0" rpy="0 0 0"/>
   </joint>
@@ -154,6 +123,6 @@
       <robotNamespace>/</robotNamespace>
       <updateRate>50.0</updateRate>
-      <bodyName>imu_link</bodyName>
-      <topicName>imu</topicName>
+      <bodyName>base_link</bodyName>
+      <topicName>imu/data</topicName>
       <accelDrift>0.005 0.005 0.005</accelDrift>
       <accelGaussianNoise>0.005 0.005 0.005</accelGaussianNoise>
@@ -167,9 +136,9 @@
     <axis xyz="1 0 0"/>
     <origin xyz="0 0 0.19"/>
-    <parent link="chassis"/>
+    <parent link="base_link"/>
     <child link="imu_link"/>
   </joint>
   <!-- Create camera instance -->
-  <xacro:realsense-rs200 prefix="" parent="chassis">
+  <xacro:realsense-rs200 prefix="" parent="base_link">
     <origin xyz="0.285 0 .065" rpy="0 0 0" />
   </xacro:realsense-rs200>
@@ -179,14 +148,14 @@
   <xacro:property name="wheel_offset_z" value="0.0" />
   <!-- Add omni wheels to the robot -->
-  <xacro:omni_wheel prefix="front_right" parent="chassis" reflect="false">
+  <xacro:omni_wheel prefix="front_right" parent="base_link" reflect="false">
     <origin xyz="${wheel_offset_x} -${wheel_offset_y} ${wheel_offset_z}" rpy="0 0 0"/>
   </xacro:omni_wheel>
-  <xacro:omni_wheel prefix="front_left" parent="chassis" reflect="true">
+  <xacro:omni_wheel prefix="front_left" parent="base_link" reflect="true">
     <origin xyz="${wheel_offset_x} ${wheel_offset_y} ${wheel_offset_z}" rpy="0 0 0"/>
   </xacro:omni_wheel>
-  <xacro:omni_wheel prefix="back_left" parent="chassis" reflect="true">
+  <xacro:omni_wheel prefix="back_left" parent="base_link" reflect="true">
     <origin xyz="-${wheel_offset_x} ${wheel_offset_y} ${wheel_offset_z}" rpy="0 0 0"/>
   </xacro:omni_wheel>
-  <xacro:omni_wheel prefix="back_right" parent="chassis" reflect="false">
+  <xacro:omni_wheel prefix="back_right" parent="base_link" reflect="false">
     <origin xyz="-${wheel_offset_x} -${wheel_offset_y} ${wheel_offset_z}" rpy="0 0 0"/>
   </xacro:omni_wheel>

Commit message: running online cartographer SLAM. Chassis is renamed to base_link in the robot description. IMU simulation is replaced with libhector_gazebo_ros_imu

File: urdf/robot.xacro (robot description, xacro)
@@ -4,8 +4,5 @@
 <xacro:include filename="$(find gazebo_simulation)/urdf/realsense-RS200.macro.xacro"/>
 <xacro:include filename="$(find gazebo_simulation)/urdf/omni_wheel.urdf.xacro" />
-  <gazebo reference="chassis">
-    <material>Gazebo/RedBright</material>
-  </gazebo>
-  <gazebo reference="chassis2">
+  <gazebo reference="base_link">
     <material>Gazebo/RedBright</material>
   </gazebo>
@@ -19,10 +16,5 @@
     https://www.expo21xx.com/industrial-robots/20317_st3_mobile-robot-research/default.htm
   -->
-  <joint name="robot_footprint_joint" type="fixed">
-    <origin xyz="0 0 0" rpy="0 0 0" />
-    <parent link="robot_footprint"/>
-    <child link="chassis" />
-  </joint>
-  <link name='chassis'>
+  <link name='base_link'>
     <pose>0 0 0.1 0 0 0</pose>
     <inertial>
@@ -41,5 +33,5 @@
       </geometry>
     </collision>
-    <visual name='chassis_visual'>
+    <visual name='base_link_visual'>
       <origin xyz="0 0 0" rpy=" 0 0 0"/>
       <geometry>
@@ -48,35 +40,12 @@
     </visual>
   </link>
-  <joint name="robot_footprint_joint2" type="fixed">
+  <joint name="robot_footprint_joint" type="fixed">
     <origin xyz="0 0 0" rpy="0 0 0" />
-    <parent link="chassis"/>
-    <child link="chassis2" />
+    <parent link="base_link" />
+    <child link="robot_footprint"/>
   </joint>
-  <link name='chassis2'>
-    <inertial>
-      <mass value="1.0"/>
-      <origin xyz="0.0 0 0" rpy=" 0 0 0"/>
-      <inertia
-          ixx="0.1" ixy="0" ixz="0"
-          iyy="0.1" iyz="0"
-          izz="0.1"
-      />
-    </inertial>
-    <collision name='collision2'>
-      <origin xyz="0 0 0" rpy=" 0 0 0"/>
-      <geometry>
-        <box size=".135 .400 .110"/>
-      </geometry>
-    </collision>
-    <visual name='chassis2_visual'>
-      <origin xyz="0 0 0" rpy=" 0 0 0"/>
-      <geometry>
-        <box size=".135 .400 .110"/>
-      </geometry>
-    </visual>
-  </link>
   <joint name="robot_lidar_platform_joint" type="fixed">
     <origin xyz="0.0 0.0 0.08" rpy="0 0 0" />
-    <parent link="chassis"/>
+    <parent link="base_link"/>
     <child link="robot_lidar_platform" />
   </joint>
@@ -97,5 +66,5 @@
       </geometry>
     </collision>
-    <visual name='chassis2_visual'>
+    <visual>
       <origin xyz="0.0 0 0" rpy=" 0 0 0"/>
       <geometry>
@@ -137,35 +106,39 @@
     <origin xyz="0.0 0.0 0.15" rpy="0 0 0"/>
     <child link="hokuyo"/>
-    <parent link="chassis"/>
+    <parent link="base_link"/>
     <axis xyz="0 1 0" rpy="0 0 0"/>
   </joint>
   <!-- IMU -->
+  <!-- from https://github.com/jackal/jackal/blob/indigo-devel/jackal_description/urdf/jackal.urdf.xacro -->
+  <xacro:property name="dummy_inertia" value="1e-09"/>
   <link name="imu_link">
     <inertial>
       <mass value="0.001"/>
-      <origin rpy="0 0 0" xyz="0 0 0"/>
-      <inertia ixx="0.0001" ixy="0" ixz="0" iyy="0.000001" iyz="0" izz="0.0001"/>
+      <origin xyz="0 0 0" rpy="0 0 0"/>
+      <inertia ixx="${dummy_inertia}" ixy="0.0" ixz="0.0" iyy="${dummy_inertia}" iyz="0.0" izz="${dummy_inertia}"/>
     </inertial>
-    <visual>
-      <origin rpy="0 0 0" xyz="0 0 0"/>
-      <geometry>
-        <box size="0.001 0.001 0.001"/>
-      </geometry>
-    </visual>
-    <collision>
-      <origin rpy="0 0 0" xyz="0 0 0"/>
-      <geometry>
-        <box size=".001 .001 .001"/>
-      </geometry>
-    </collision>
   </link>
+  <gazebo>
+    <plugin name="imu_controller" filename="libhector_gazebo_ros_imu.so">
+      <robotNamespace>/</robotNamespace>
+      <updateRate>50.0</updateRate>
+      <bodyName>base_link</bodyName>
+      <topicName>imu/data</topicName>
+      <accelDrift>0.005 0.005 0.005</accelDrift>
+      <accelGaussianNoise>0.005 0.005 0.005</accelGaussianNoise>
+      <rateDrift>0.005 0.005 0.005 </rateDrift>
+      <rateGaussianNoise>0.005 0.005 0.005 </rateGaussianNoise>
+      <headingDrift>0.005</headingDrift>
+      <headingGaussianNoise>0.005</headingGaussianNoise>
+    </plugin>
+  </gazebo>
   <joint name="imu_joint" type="fixed">
     <axis xyz="1 0 0"/>
     <origin xyz="0 0 0.19"/>
-    <parent link="chassis"/>
+    <parent link="base_link"/>
     <child link="imu_link"/>
   </joint>
   <!-- Create camera instance -->
-  <xacro:realsense-rs200 prefix="" parent="chassis">
+  <xacro:realsense-rs200 prefix="" parent="base_link">
     <origin xyz="0.285 0 .065" rpy="0 0 0" />
   </xacro:realsense-rs200>
@@ -175,14 +148,14 @@
   <xacro:property name="wheel_offset_z" value="0.0" />
   <!-- Add omni wheels to the robot -->
-  <xacro:omni_wheel prefix="front_right" parent="chassis" reflect="false">
+  <xacro:omni_wheel prefix="front_right" parent="base_link" reflect="false">
     <origin xyz="${wheel_offset_x} -${wheel_offset_y} ${wheel_offset_z}" rpy="0 0 0"/>
   </xacro:omni_wheel>
-  <xacro:omni_wheel prefix="front_left" parent="chassis" reflect="true">
+  <xacro:omni_wheel prefix="front_left" parent="base_link" reflect="true">
     <origin xyz="${wheel_offset_x} ${wheel_offset_y} ${wheel_offset_z}" rpy="0 0 0"/>
   </xacro:omni_wheel>
-  <xacro:omni_wheel prefix="back_left" parent="chassis" reflect="true">
+  <xacro:omni_wheel prefix="back_left" parent="base_link" reflect="true">
     <origin xyz="-${wheel_offset_x} ${wheel_offset_y} ${wheel_offset_z}" rpy="0 0 0"/>
   </xacro:omni_wheel>
-  <xacro:omni_wheel prefix="back_right" parent="chassis" reflect="false">
+  <xacro:omni_wheel prefix="back_right" parent="base_link" reflect="false">
     <origin xyz="-${wheel_offset_x} -${wheel_offset_y} ${wheel_offset_z}" rpy="0 0 0"/>
   </xacro:omni_wheel>

Commit message: roll back chassis2

File: urdf/robot.xacro (robot description, xacro)
@@ -5,4 +5,7 @@
 <xacro:include filename="$(find gazebo_simulation)/urdf/omni_wheel.urdf.xacro" />
   <gazebo reference="base_link">
+    <material>Gazebo/RedBright</material>
+  </gazebo>
+  <gazebo reference="chassis2">
     <material>Gazebo/RedBright</material>
   </gazebo>
@@ -44,4 +47,32 @@
     <parent link="base_link" />
     <child link="robot_footprint"/>
+  </joint>
+  <link name='chassis2'>
+    <inertial>
+      <mass value="1.0"/>
+      <origin xyz="0.0 0 0" rpy=" 0 0 0"/>
+      <inertia
+              ixx="0.1" ixy="0" ixz="0"
+              iyy="0.1" iyz="0"
+              izz="0.1"
+      />
+    </inertial>
+    <collision name='collision2'>
+      <origin xyz="0 0 0" rpy=" 0 0 0"/>
+      <geometry>
+        <box size=".135 .400 .110"/>
+      </geometry>
+    </collision>
+    <visual name='chassis2_visual'>
+      <origin xyz="0 0 0" rpy=" 0 0 0"/>
+      <geometry>
+        <box size=".135 .400 .110"/>
+      </geometry>
+    </visual>
+  </link>
+  <joint name="robot_footprint_joint2" type="fixed">
+    <origin xyz="0 0 0" rpy="0 0 0" />
+    <parent link="base_link"/>
+    <child link="chassis2" />
   </joint>
   <joint name="robot_lidar_platform_joint" type="fixed">
